File: conferenceCallPCB.sch (KiCad schematic (older format))
At the start: 2 parts

Commit message: Continued working on schematic
Parts:
- added C? (x3): 100nF, Capacitor_SMD:C_0603_1608Metric_Pad1.08x0.95mm_HandSolder, symbol Device:C
- added C?: 4.7uF, Capacitor_SMD:C_0603_1608Metric_Pad1.08x0.95mm_HandSolder, symbol Device:C
- added C? (x2): 12pF, Capacitor_SMD:C_0603_1608Metric_Pad1.08x0.95mm_HandSolder, symbol Device:C
- added C?: 1.0uF, Capacitor_SMD:C_0603_1608Metric_Pad1.08x0.95mm_HandSolder, symbol Device:C
- added C?: 100pF, Capacitor_SMD:C_0603_1608Metric_Pad1.08x0.95mm_HandSolder, symbol Device:C
- added C?: N.C., Capacitor_SMD:C_0603_1608Metric_Pad1.08x0.95mm_HandSolder, symbol Device:C
- added C?: 0.8pF, Capacitor_SMD:C_0603_1608Metric_Pad1.08x0.95mm_HandSolder, symbol Device:C
- added L?: 3.9nH, Inductor_SMD:L_0402_1005Metric_Pad0.77x0.64mm_HandSolder, symbol Device:L
- added Y?: Crystal, Crystal:Crystal_SMD_2012-2Pin_2.0x1.2mm_HandSoldering, symbol Device:Crystal
Connections:
- net GND: now also U?.31 (VSS), U?.45 (VSS), U?.49 (VSS), C?.1, C?.1, C?.2, C?.2, C?.2, C?.2, C?.2, C?.2, C?.2, C?.2
- net at U?.1 (DEC1): now also C?.1
- net +3V3: now reaches U?.13 (VDD), U?.36 (VDD), U?.48 (VDD)
- net +3V3: now also C?.1, C?.1, C?.1
- net at U?.30 (ANT): now also C?.1, L?.2
- net at U?.32 (DEC2): now also C?.1
- net at U?.33 (DEC3): now also C?.1
- net at U?.34 (XC1): now also C?.2, Y?.2
- net at U?.35 (XC2): now also C?.2, Y?.1
- net DEC4: now reaches U?.46 (DEC4)
- net DEC4: now also U?.47 (DCC), C?.1
- new net RF: L?.1
